File: pcbStuff/shrine/hope/hope.kicad_pcb (KiCad board)
At the start: 2 copper layers, 14 parts, among them U1 LM555xN, U2 74LS74, U3 74LS74, U4 74LS74

Commit message: done???
Parts:
- BT1, D4, D5, R1, R2, U1: moved to B.Cu
- moved D3 156.8 mm to (54.7, 132.8)
- moved D4 105.5 mm to (118.0, 152.3), turned to 90 degrees
- moved U4 71.7 mm to (79.0, 104.2)
- moved U3 63.0 mm to (79.0, 84.5)
- moved U1 60.1 mm to (105.8, 114.9), turned to 180 degrees
- moved R2 59.9 mm to (105.8, 127.2), turned to 180 degrees
- moved R3 53.8 mm to (110.8, 127.3), turned to 90 degrees
- moved C1 46.8 mm to (114.0, 116.4), turned to 90 degrees
- moved D5 45.8 mm to (157.8, 100.0), turned to 180 degrees
- moved BT1 41.6 mm to (101.5, 101.2), turned to 180 degrees
- moved D2 40.4 mm to (55.5, 67.8)
- moved R1 35.3 mm to (127.1, 109.0), turned to 180 degrees
- moved D1 22.2 mm to (118.2, 45.7), turned to -90 degrees
- moved U2 18.5 mm to (116.4, 87.4)
Routing:
- net Net-(D1-K): track 0.00 -> 396.7 mm
- net Net-(U1-Q): track 0.00 -> 126.0 mm
- net Net-(D3-A): track 0.00 -> 120.7 mm
- net Net-(BT1-+): track 0.00 -> 105.8 mm, vias 0 -> 1
- net Net-(BT1--): track 0.00 -> 102.1 mm, vias 0 -> 1
- net Net-(D4-A): track 0.00 -> 101.6 mm, vias 0 -> 1
- net Net-(D5-A): track 0.00 -> 87.7 mm, vias 0 -> 1
- net Net-(D2-A): track 0.00 -> 60.4 mm
- net Net-(D1-A): track 0.00 -> 55.3 mm
- net Net-(U1-DIS): track 0.00 -> 25.6 mm
- net Net-(U1-THR): track 0.00 -> 19.2 mm
Other:
- board outline added: 119.7 x 125.8 mm

Commit message: math
Parts:
- BT1, D4, D5, R1, R2, U1: moved to F.Cu
- moved D2 120.0 mm to (166.1, 114.3), turned to -162 degrees
- moved U1 112.9 mm to (49.0, 17.3), turned to 0 degrees
- moved C1 106.2 mm to (49.8, 31.8), turned to 0 degrees
- moved U2 104.0 mm to (24.2, 39.4)
- moved D3 100.3 mm to (151.2, 160.3), turned to 126 degrees
- moved BT1 100.2 mm to (35.0, 26.3), turned to 0 degrees
- moved R1 99.2 mm to (56.5, 39.3), turned to 0 degrees
- moved R2 97.3 mm to (56.5, 43.4), turned to 0 degrees
- moved R3 96.6 mm to (56.5, 47.4), turned to 0 degrees
- moved U4 72.9 mm to (45.7, 39.4)
- moved D5 71.3 mm to (87.9, 114.3), turned to -18 degrees
- moved U3 63.0 mm to (34.9, 39.4)
- moved D1 39.1 mm to (127.0, 83.8)
- moved D4 17.1 mm to (102.8, 160.3), turned to 54 degrees
Routing:
- net Net-(D1-K): track 396.7 -> 0.00 mm
- net Net-(U1-Q): track 126.0 -> 0.00 mm
- net Net-(D3-A): track 120.7 -> 0.00 mm
- net Net-(BT1-+): track 105.8 -> 0.00 mm, vias 1 -> 0
- net Net-(BT1--): track 102.1 -> 0.00 mm, vias 1 -> 0
- net Net-(D4-A): track 101.6 -> 0.00 mm, vias 1 -> 0
- net Net-(D5-A): track 87.7 -> 0.00 mm, vias 1 -> 0
- net Net-(D2-A): track 60.4 -> 0.00 mm
- net Net-(D1-A): track 55.3 -> 0.00 mm
- net Net-(U1-DIS): track 25.6 -> 0.00 mm
- net Net-(U1-THR): track 19.2 -> 0.00 mm
Other:
- board size 119.7 x 125.8 mm -> 96.6 x 91.9 mm
