File: pcbStuff/potato/v1/RAM/RAM.kicad_pcb (KiCad board)
At the start: 2 copper layers, 17 parts, among them U1 74LS138, U10 74LS74, U11 74LS74, U12 74LS00, U13 74LS74, U14 74LS00, U15 74LS74, U16 74LS74, U2 74LS138, U3 74LS04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

Commit message: THE FUCK YOU MEAN 1.27
Parts:
- U2: moved to F.Cu
- moved U1 197.2 mm to (41.6, 64.8), turned to 0 degrees
- moved U2 183.1 mm to (52.4, 64.8), turned to 0 degrees
- moved U3 171.2 mm to (41.6, 21.4), turned to 0 degrees
- moved 6-1 144.9 mm to (45.0, 62.0)
- moved U15 83.7 mm to (95.5, 40.7), turned to 0 degrees
- moved U16 81.7 mm to (106.3, 40.7), turned to 0 degrees
- moved U10 71.0 mm to (115.6, 85.1)
- moved U4 60.8 mm to (176.7, 131.9)
- moved U14 57.6 mm to (84.7, 40.7)
- moved U9 53.0 mm to (100.3, 77.5)
- moved U7 49.3 mm to (163.0, 116.5)
- moved U11 46.1 mm to (115.6, 100.3)
- moved U5 39.9 mm to (176.7, 117.9)
- moved U12 30.9 mm to (100.3, 100.3)
- moved U6 26.9 mm to (176.7, 103.4)
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Routing:
- net Net-(U1-O5): track 140.8 -> 0.00 mm, vias 6 -> 0
- net Net-(U11B-D): track 229.6 -> 119.4 mm, vias 4 -> 6
- net Net-(U10A-D): track 218.4 -> 115.3 mm, vias 2 -> 6
- net Net-(U5B-~{Q}): track 0.00 -> 84.2 mm, vias 0 -> 2
- net Net-(U4B-~{Q}): track 0.00 -> 77.8 mm, vias 0 -> 2
- net Net-(U6A-~{Q}): track 0.00 -> 73.6 mm, vias 0 -> 2
- net Net-(U10B-D): track 62.9 -> 123.9 mm, vias 2 -> 8
- net Net-(U12-Pad12): track 144.7 -> 86.1 mm, vias 0 -> 4
- net Net-(U4A-C): track 0.00 -> 58.4 mm, vias 0 -> 2
- net Net-(U5A-~{Q}): track 0.00 -> 58.4 mm, vias 0 -> 2
- net Net-(U5B-C): track 0.00 -> 58.0 mm
- net Net-(U6B-~{Q}): track 0.00 -> 57.5 mm, vias 0 -> 2
- net Net-(U15B-~{Q}): track 52.8 -> 0.00 mm, vias 2 -> 0
- net Net-(U1-GND): track 139.6 -> 190.8 mm, vias 2 -> 4
- net Net-(U15A-C): track 49.1 -> 0.00 mm, vias 3 -> 0
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
Commit message: im confused
Parts:
- moved U16 138.7 mm to (186.7, 153.7), turned to 90 degrees
- moved U3 135.9 mm to (158.8, 90.2)
- moved U15 135.5 mm to (186.7, 141.0), turned to 90 degrees
- moved U14 128.8 mm to (171.4, 135.9)
- moved U1 118.9 mm to (158.8, 44.5)
- moved 6-1 115.8 mm to (151.9, 106.7), turned to 90 degrees
- moved U2 106.4 mm to (158.8, 67.3)
- moved U10 72.2 mm to (186.7, 97.8)
- moved U11 72.2 mm to (186.7, 113.0)
- moved U13 72.2 mm to (186.7, 128.3)
- moved U12 72.2 mm to (171.4, 113.0)
- moved U9 72.2 mm to (171.4, 90.2)
- moved U6 52.3 mm to (186.7, 52.1)
- moved U8 52.2 mm to (171.4, 44.5)
- moved U5 51.6 mm to (186.7, 67.3)
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Routing:
- net Net-(U1-E1): track 142.9 -> 309.1 mm
- net Net-(U10A-D): track 115.3 -> 269.0 mm, vias 6 -> 5
- net Net-(U10B-D): track 123.9 -> 236.8 mm, vias 8 -> 2
- net Net-(U1-GND): track 190.8 -> 294.7 mm
- net Net-(U15B-~{Q}): track 0.00 -> 52.8 mm
- net Net-(U15A-C): track 0.00 -> 51.1 mm, vias 0 -> 2
- net Net-(U11B-D): track 119.4 -> 169.4 mm, vias 6 -> 5
- net Net-(U11B-~{Q}): track 0.00 -> 45.9 mm, vias 0 -> 1
- net Net-(U13B-~{Q}): track 0.00 -> 43.1 mm, vias 0 -> 1
- net Net-(U5B-~{Q}): track 84.2 -> 45.9 mm, vias 2 -> 1
- net Net-(U6A-~{Q}): track 73.6 -> 35.3 mm, vias 2 -> 1
- net Net-(U11A-C): track 0.00 -> 35.7 mm, vias 0 -> 1
- net Net-(U10A-~{Q}): track 0.00 -> 35.3 mm, vias 0 -> 1
- net Net-(U4B-~{Q}): track 77.8 -> 43.1 mm, vias 2 -> 1
- net Net-(U15A-~{Q}): track 0.00 -> 33.2 mm
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Other:
- board outline added: 52.4 x 116.8 mm

Commit message: oh my dear god
Routing:
- net Net-(U1-O3): track 9.72 -> 95.2 mm, vias 1 -> 0
- net Net-(U1-O5): track 18.4 -> 93.2 mm, vias 1 -> 2
- net Net-(U1-E1): track 309.1 -> 382.3 mm, vias 2 -> 3
- net Net-(U1-GND): track 294.7 -> 349.2 mm
- net /strobe: track 0.00 -> 53.5 mm, vias 0 -> 1
- net Net-(U2-O5): track 19.4 -> 72.8 mm, vias 0 -> 2
- net Net-(U1-A0): track 0.00 -> 37.5 mm
- net Net-(U12-Pad12): track 108.7 -> 145.8 mm, vias 0 -> 3
- net Net-(U1-O4): track 9.72 -> 43.1 mm
- net Net-(U1-O7): track 18.4 -> 51.3 mm, vias 1 -> 3
- net Net-(U1-A1): track 0.00 -> 30.6 mm, vias 0 -> 1
- net Net-(U2-A2): track 0.00 -> 29.8 mm, vias 0 -> 3
- net Net-(U1-A2): track 0.00 -> 22.8 mm, vias 0 -> 1
- net Net-(U2-A1): track 0.00 -> 22.2 mm, vias 0 -> 3
- net Net-(U1-O6): track 11.0 -> 32.9 mm
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
Commit message: i am fucking lossing it
Routing:
- net Net-(U11B-D): track 170.5 -> 274.1 mm, vias 5 -> 12
- net Net-(U10A-D): track 252.8 -> 311.0 mm, vias 7 -> 9
- net Net-(U1-GND): track 349.2 -> 392.1 mm
- net Net-(U12-Pad12): track 145.8 -> 177.3 mm
- net Net-(U10B-D): track 250.9 -> 267.6 mm, vias 5 -> 7
- net Net-(6-1-Pad3): track 13.2 -> 0.00 mm
- net Net-(U2-O5): track 72.8 -> 65.5 mm
- net Net-(U2-O3): track 13.3 -> 19.4 mm
- net Net-(U1-O5): track 93.2 -> 98.2 mm
- net Net-(U1-O3): track 95.2 -> 99.7 mm, vias 0 -> 2
- net Net-(U1-E1): track 382.3 -> 383.8 mm
