File: pcbStuff/potato/v1/RAM/RAM.kicad_pcb (KiCad board)
At the start: 2 copper layers, 52.4 x 116.8 mm, 17 parts, among them U1 74LS138, U10 74LS74, U11 74LS74, U12 74LS00, U13 74LS74, U14 74LS00, U15 74LS74, U16 74LS74, U2 74LS138, U3 74LS04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

Commit message: ass cancer
name by armando
Parts:
- moved U3 75.0 mm to (194.3, 24.1)
- moved U2 57.1 mm to (189.2, 19.1), turned to -90 degrees
- moved 6-1 36.1 mm to (123.9, 83.9)
- moved U1 33.0 mm to (189.2, 31.8), turned to -90 degrees
Routing:
- net Net-(U10B-D): track 236.8 -> 155.3 mm
- net /strobe: track 0.00 -> 62.7 mm, vias 0 -> 3
- net Net-(U1-E1): track 309.1 -> 361.0 mm, vias 2 -> 4
- net Net-(U12-Pad12): track 108.7 -> 150.9 mm, vias 0 -> 2
- net Net-(U2-A0): track 0.00 -> 37.7 mm
- net Net-(U1-A0): track 0.00 -> 37.7 mm
- net Net-(U10A-D): track 269.0 -> 233.6 mm, vias 5 -> 15
- net Net-(U1-A1): track 0.00 -> 34.6 mm
- net Net-(U2-A1): track 0.00 -> 34.6 mm
- net Net-(U2-A2): track 0.00 -> 31.5 mm
- net Net-(U1-A2): track 0.00 -> 31.5 mm
- net Net-(6-1-Pad3): track 13.9 -> 42.8 mm
- net Net-(U2-O3): track 13.3 -> 30.7 mm
- net Net-(U1-GND): track 294.7 -> 306.2 mm, vias 4 -> 3
- net Net-(U1-O3): track 9.72 -> 20.7 mm, vias 1 -> 0
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Other:
- board size 52.4 x 116.8 mm -> 55.9 x 139.7 mm

Commit message: only 5 remain
Parts:
- moved 6-1 36.8 mm to (160.8, 83.9)
Routing:
- net Net-(U2-O3): track 30.7 -> 149.8 mm, vias 1 -> 5
- net Net-(U1-O3): track 20.7 -> 125.1 mm, vias 0 -> 1
- net Net-(U2-O5): track 26.8 -> 121.5 mm, vias 0 -> 2
- net Net-(U1-O5): track 24.5 -> 118.7 mm, vias 1 -> 2
- net Net-(U11B-D): track 171.5 -> 263.8 mm, vias 5 -> 13
- net Net-(U10B-D): track 155.3 -> 229.3 mm, vias 2 -> 9
- net Net-(U2-O4): track 29.4 -> 99.9 mm, vias 0 -> 3
- net Net-(U1-O7): track 24.5 -> 82.1 mm, vias 1 -> 3
- net Net-(U1-O4): track 18.4 -> 75.9 mm, vias 0 -> 2
- net Net-(U2-O7): track 25.6 -> 81.8 mm, vias 0 -> 2
- net Net-(6-1-Pad3): track 42.8 -> 96.8 mm, vias 1 -> 3
- net Net-(U10A-D): track 233.6 -> 263.3 mm, vias 15 -> 16
- net Net-(U1-E1): track 361.0 -> 387.9 mm
- net Net-(U2-O6): track 23.3 -> 41.6 mm, vias 0 -> 1
- net Net-(U1-A0): track 37.7 -> 51.0 mm, vias 0 -> 1
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Other:
- board size 55.9 x 139.7 mm -> 43.5 x 139.7 mm

Commit message: 2 LIttlE FUCKERS
Routing:
- net Net-(U1-E1): track 387.9 -> 475.2 mm
- net Net-(U10B-D): track 229.3 -> 286.9 mm, vias 9 -> 10
- net Net-(U1-GND): track 306.0 -> 344.2 mm, vias 3 -> 4
- net Net-(U15A-C): track 51.1 -> 35.7 mm
- net Net-(U1-O4): track 75.9 -> 74.2 mm
- net Net-(U1-O3): track 125.1 -> 124.1 mm, vias 1 -> 5
- net Net-(U2-O4): track 99.9 -> 99.1 mm
- net Net-(U2-O5): track 121.5 -> 122.3 mm
- net Net-(U12-Pad12): track 150.1 -> 149.4 mm
- net Net-(U10A-D): track 263.3 -> 262.5 mm
- net Net-(U1-O5): vias 2 -> 4
- net Net-(U1-O7): vias 3 -> 1

Commit message: why is it impossible
Routing:
- net Net-(U1-GND): track 344.2 -> 351.6 mm, vias 4 -> 5
- net Net-(U1-E1): track 475.2 -> 480.3 mm, vias 4 -> 5
- net Net-(6-1-Pad3): vias 3 -> 4
- net /strobe: vias 5 -> 3
Changed lines of the file:
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@@
+	)
+	(via
+		(at 177.8 29.21)
+		(size 0.6)
+		(drill 0.3)
+		(layers "F.Cu" "B.Cu")
+		(net 3)
 	)
 	(via
@@
 	)
 	(segment
+		(start 171.45 31.755)
+		(end 173.995 29.21)
+		(width 0.2)
+		(layer "B.Cu")
+		(net 3)
+	)
+	(segment
 		(start 204.47 110.49)
 		(end 204.47 100.33)
@@
 	)
 	(segment
+		(start 173.995 29.21)
+		(end 177.8 29.21)
+		(width 0.2)
+		(layer "B.Cu")
+		(net 3)
+	)
+	(segment
 		(start 204.47 80.01)
 		(end 204.47 69.85)
@@
 	)
 	(segment
-		(start 184.155 29.21)
-		(end 186.695 29.21)
-		(width 0.2)
-		(layer "F.Cu")
-		(net 4)
-	)
-	(segment
 		(start 203.2 115.57)
 		(end 204.47 116.84)
@@
 	)
 	(segment
+		(start 189.23 26.675)
+		(end 189.23 27.94)
+		(width 0.2)
+		(layer "F.Cu")
+		(net 4)
+	)
+	(segment
 		(start 189.23 148.59)
 		(end 186.69 146.05)
@@
 	)
 	(segment
-		(start 186.695 29.21)
-		(end 189.23 26.675)
-		(width 0.2)
-		(layer "F.Cu")
-		(net 4)
-	)
-	(segment
 		(start 189.23 46.99)
 		(end 186.69 44.45)
@@
 	)
 	(segment
-		(start 181.61 31.755)
-		(end 184.155 29.21)
-		(width 0.2)
-		(layer "F.Cu")
-		(net 4)
-	)
-	(segment
 		(start 204.47 101.6)
 		(end 204.47 90.17)
@@
 	)
 	(segment
+		(start 189.23 27.94)
+		(end 190.501397 29.211397)
+		(width 0.2)
+		(layer "F.Cu")
+		(net 4)
+	)
+	(segment
 		(start 182.88 73.671207)
 		(end 182.88 73.66)
@@
 	)
 	(via
+		(at 190.501397 29.211397)
+		(size 0.6)
+		(drill 0.3)
+		(layers "F.Cu" "B.Cu")
+		(net 4)
+	)
+	(via
 		(at 191.771397 40.641397)
 		(size 0.6)
@@
 		(drill 0.3)
 		(layers "F.Cu" "B.Cu")
+		(net 4)
+	)
+	(segment
+		(start 191.77 30.48)
+		(end 191.77 34.29)
+		(width 0.2)
+		(layer "B.Cu")
+		(net 4)
+	)
+	(segment
+		(start 189.23 36.83)
+		(end 189.23 39.375)
+		(width 0.2)
+		(layer "B.Cu")
 		(net 4)
 	)
@@
 	)
 	(segment
+		(start 190.501397 29.211397)
+		(end 191.77 30.48)
+		(width 0.2)
+		(layer "B.Cu")
+		(net 4)
+	)
+	(segment
 		(start 186.69 120.65)
 		(end 186.69 118.11)
@@
 	)
 	(segment
+		(start 191.77 34.29)
+		(end 189.23 36.83)
+		(width 0.2)
+		(layer "B.Cu")
+		(net 4)
+	)
+	(segment
 		(start 195.58 41.912794)
 		(end 193.042794 41.912794)
@@
 	)
 	(segment
+		(start 191.77 38.1)
+		(end 191.77 26.67)
+		(width 0.2)
+		(layer "F.Cu")
+		(net 7)
+	)
+	(segment
+		(start 191.77 26.67)
+		(end 194.31 24.13)
+		(width 0.2)
+		(layer "F.Cu")
+		(net 7)
+	)
+	(segment
 		(start 171.457794 41.917794)
 		(end 171.45 41.91)
@@
 	)
 	(via
+		(at 191.77 38.1)
+		(size 0.6)
+		(drill 0.3)
+		(layers "F.Cu" "B.Cu")
+		(net 7)
+	)
+	(via
 		(at 170.178603 41.911397)
 		(size 0.6)
@@
 	)
 	(segment
-		(start 191.77 26.67)
-		(end 191.77 39.37)
-		(width 0.2)
-		(layer "B.Cu")
-		(net 7)
-	)
-	(segment
 		(start 162.56 35.555793)
 		(end 162.56 60.96)
@@
 	)
 	(segment
-		(start 194.31 24.13)
-		(end 191.77 26.67)
+		(start 191.77 39.37)
+		(end 191.77 38.1)
 		(width 0.2)
 		(layer "B.Cu")
@@
 	)
 	(segment
-		(start 189.23 24.13)
-		(end 187.96 24.13)
-		(width 0.2)
-		(layer "F.Cu")
-		(net 10)
-	)
-	(segment
 		(start 165.1 25.4)
 		(end 162.56 22.86)
@@
 	)
 	(segment
+		(start 176.53 31.755)
+		(end 179.07 31.755)
+		(width 0.2)
+		(layer "F.Cu")
+		(net 10)
+	)
+	(segment
+		(start 176.53 19.055)
+		(end 179.07 19.055)
+		(width 0.2)
+		(layer "F.Cu")
+		(net 10)
+	)
+	(segment
+		(start 175.26 22.86)
+		(end 167.64 22.86)
+		(width 0.2)
+		(layer "F.Cu")
+		(net 10)
+	)
+	(segment
+		(start 185.4175 24.135294)
+		(end 184.150294 24.135294)
+		(width 0.2)
+		(layer "F.Cu")
+		(net 10)
+	)
+	(segment
+		(start 175.265 22.86)
+		(end 175.26 22.86)
+		(width 0.2)
+		(layer "F.Cu")
+		(net 10)
+	)
+	(segment
+		(start 162.56 22.86)
+		(end 158.75 22.86)
+		(width 0.2)
+		(layer "F.Cu")
+		(net 10)
+	)
+	(via
+		(at 167.64 25.4)
+		(size 0.6)
+		(drill 0.3)
+		(layers "F.Cu" "B.Cu")
+		(net 10)
+	)
+	(via
+		(at 185.4175 24.135294)
+		(size 0.6)
+		(drill 0.3)
+		(layers "F.Cu" "B.Cu")
+		(net 10)
+	)
+	(via
+		(at 165.1 25.4)
+		(size 0.6)
+		(drill 0.3)
+		(layers "F.Cu" "B.Cu")
+		(net 10)
+	)
+	(segment
+		(start 185.42 24.132794)
+		(end 185.4175 24.135294)
+		(width 0.2)
+		(layer "B.Cu")
+		(net 10)
+	)
+	(segment
+		(start 185.422794 24.13)
+		(end 185.4175 24.135294)
+		(width 0.2)
+		(layer "B.Cu")
+		(net 10)
+	)
+	(segment
+		(start 189.23 24.13)
+		(end 185.422794 24.13)
+		(width 0.2)
+		(layer "B.Cu")
+		(net 10)
+	)
+	(segment
+		(start 185.42 24.13)
+		(end 185.42 24.132794)
+		(width 0.2)
+		(layer "B.Cu")
+		(net 10)
+	)
+	(segment
 		(start 189.23 29.21)
 		(end 191.77 26.67)
 		(width 0.2)
-		(layer "F.Cu")
+		(layer "B.Cu")
 		(net 10)
 	)
 	(segment
-		(start 176.53 31.755)
-		(end 179.07 31.755)
-		(width 0.2)
-		(layer "F.Cu")
+		(start 181.615 29.21)
+		(end 189.23 29.21)
+		(width 0.2)
+		(layer "B.Cu")
 		(net 10)
 	)
 	(segment
-		(start 176.53 19.055)
-		(end 179.07 19.055)
-		(width 0.2)
-		(layer "F.Cu")
-		(net 10)
-	)
-	(segment
-		(start 175.26 22.86)
-		(end 167.64 22.86)
-		(width 0.2)
-		(layer "F.Cu")
+		(start 179.07 31.755)
+		(end 181.615 29.21)
+		(width 0.2)
+		(layer "B.Cu")
 		(net 10)
 	)
@@
 		(end 189.23 24.13)
 		(width 0.2)
-		(layer "F.Cu")
-		(net 10)
-	)
-	(segment
-		(start 185.4175 24.135294)
-		(end 184.150294 24.135294)
-		(width 0.2)
-		(layer "F.Cu")
-		(net 10)
-	)
-	(segment
-		(start 175.265 22.86)
-		(end 175.26 22.86)
-		(width 0.2)
-		(layer "F.Cu")
-		(net 10)
-	)
-	(segment
-		(start 162.56 22.86)
-		(end 158.75 22.86)
-		(width 0.2)
-		(layer "F.Cu")
-		(net 10)
-	)
-	(via
-		(at 167.64 25.4)
-		(size 0.6)
-		(drill 0.3)
-		(layers "F.Cu" "B.Cu")
-		(net 10)
-	)
-	(via
-		(at 189.23 29.21)
-		(size 0.6)
-		(drill 0.3)
-		(layers "F.Cu" "B.Cu")
-		(net 10)
-	)
-	(via
-		(at 185.4175 24.135294)
-		(size 0.6)
-		(drill 0.3)
-		(layers "F.Cu" "B.Cu")
-		(net 10)
-	)
-	(via
-		(at 187.96 24.13)
-		(size 0.6)
-		(drill 0.3)
-		(layers "F.Cu" "B.Cu")
-		(net 10)
-	)
-	(via
-		(at 165.1 25.4)
-		(size 0.6)
-		(drill 0.3)
-		(layers "F.Cu" "B.Cu")
-		(net 10)
-	)
-	(segment
-		(start 179.07 31.755)
-		(end 181.615 29.21)
-		(width 0.2)
-		(layer "B.Cu")
-		(net 10)
-	)
-	(segment
-		(start 185.422794 24.13)
-		(end 185.4175 24.135294)
-		(width 0.2)
-		(layer "B.Cu")
-		(net 10)
-	)
-	(segment
-		(start 185.42 24.132794)
-		(end 185.4175 24.135294)
-		(width 0.2)
-		(layer "B.Cu")
-		(net 10)
-	)
-	(segment
-		(start 187.96 24.13)
-		(end 185.422794 24.13)
-		(width 0.2)
-		(layer "B.Cu")
-		(net 10)
-	)
-	(segment
-		(start 185.42 24.13)
-		(end 185.42 24.132794)
-		(width 0.2)
-		(layer "B.Cu")
-		(net 10)
-	)
-	(segment
-		(start 181.615 29.21)
-		(end 189.23 29.21)
-		(width 0.2)
-		(layer "B.Cu")
+		(layer "B.Cu")
