File: pcbStuff/potato/v1/RAM/RAM.kicad_pcb (KiCad board)
At the start: 2 copper layers, 43.5 x 139.7 mm, 17 parts, among them U1 74LS138, U10 74LS74, U11 74LS74, U12 74LS00, U13 74LS74, U14 74LS00, U15 74LS74, U16 74LS74, U2 74LS138, U3 74LS04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

Commit message: truly a pcb of all time
Routing:
- net Net-(U1-GND): track 351.6 -> 454.2 mm, vias 5 -> 13
- net Net-(U1-A0): track 51.0 -> 57.1 mm
- net Net-(6-1-Pad3): track 96.8 -> 102.5 mm
- net Net-(U2-O5): track 122.3 -> 127.6 mm
- net /strobe: track 61.2 -> 65.3 mm
- net Net-(U2-O3): track 149.8 -> 153.0 mm
- net Net-(U2-O7): track 81.8 -> 84.9 mm
- net Net-(U2-A0): track 43.3 -> 45.9 mm
- net Net-(U1-A2): track 38.2 -> 40.2 mm
- net Net-(U10B-D): track 286.9 -> 288.8 mm
- net Net-(U1-A1): track 45.0 -> 46.0 mm
- net Net-(U1-E1): track 480.3 -> 481.3 mm, vias 5 -> 4
- net Net-(U2-O4): track 99.1 -> 100.2 mm
- net Net-(U2-O6): track 41.6 -> 42.7 mm
