File: pcbStuff/potato/v1/goodRAM/goodRAM.kicad_sch (KiCad schematic)
At the start: 0 parts

Commit message: something
Parts:
- added U1, U2: 74HC238, symbol 74xx:74HC238
- added U10, U12, U14, U15, U4, U5, U7, U9: 74LS74, symbol 74xx:74LS74
- added U11, U13, U3, U6, U8: 74LS08, symbol 74xx:74LS08
Connections:
- new net: U2.11 (Y4), U6.10, U6.2, U6.5
- new net: U10.12 (D), U10.2 (D), U11.8, U13.8, U15.2 (D), U3.8, U5.12 (D), U5.2 (D), U6.8, U8.8
- new net: U5.9 (Q), U6.9
- new net: U8.1, U9.5 (Q)
- new net: U2.9 (Y6), U8.10, U8.2, U8.5
- new net: U11.3, U12.2 (D), U13.3, U14.2 (D), U3.3, U4.2 (D), U6.3, U7.2 (D), U8.3, U9.2 (D)
- new net: U13.4, U14.9 (Q)
- new net: U13.10, U13.2, U13.5, U2.7 (Y7)
- new net: U11.6, U12.12 (D), U13.6, U14.12 (D), U3.6, U4.12 (D), U6.6, U7.12 (D), U8.6, U9.12 (D)
- new net: U6.1, U7.5 (Q)
- new net: U10.11 (C), U8.11, U9.11 (C), U9.3 (C)
- new net: U11.12, U13.12, U3.12, U6.12, U8.12
- new net: U1.9 (Y6), U8.13
- new net: U13.11, U14.11 (C), U14.3 (C), U15.3 (C)
- new net: U13.1, U14.5 (Q)
- new net: U8.4, U9.9 (Q)
- new net: U13.9, U15.5 (Q)
- new net: U5.11 (C), U6.11, U7.11 (C), U7.3 (C)
- new net: U11.4, U12.9 (Q)
- new net: U11.10, U11.2, U11.5, U2.10 (Y5)
- new net: U2.12 (Y3), U3.10, U3.2, U3.5
- new net: U3.11, U4.11 (C), U4.3 (C), U5.3 (C)
- new net: U1.12 (Y3), U3.13
- new net: U1.11 (Y4), U6.13
- new net: U3.1, U4.5 (Q)
- new net: U1.7 (Y7), U13.13
- new net: U10.3 (C), U11.11, U12.11 (C), U12.3 (C)
- new net: U1.10 (Y5), U11.13
- new net: U3.9, U5.5 (Q)
- new net: U11.1, U12.5 (Q)
- new net: U10.5 (Q), U11.9
- new net: U6.4, U7.9 (Q)
- new net: U10.9 (Q), U8.9
- new net: U3.4, U4.9 (Q)

Commit message: complement!
Parts:
- added 6-9(nice)1: ~, Connector_PinHeader_2.54mm:PinHeader_1x15_P2.54mm_Vertical, symbol PotatoComputerV1:6-9 Connector (nice)
- U1, U2: footprint (none) -> Package_DIP:DIP-16_W7.62mm
- U10, U11, U12, U13, U14, U15, U3, U4, U5, U6, U7, U8, U9: footprint (none) -> Package_DIP:DIP-14_W7.62mm
Connections:
- net at U10.12 (D), U10.2 (D), U11.8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: now also 6-9(nice)1.6 (Bus_3)
- net at U11.3, U12.2 (D), U13.3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: now also 6-9(nice)1.4 (Bus_1)
- net at U11.6, U12.12 (D), U13.6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: now also 6-9(nice)1.5 (Bus_2)
- net VCC: now reaches U5.14 (VCC)
- net VCC: now also U1.16 (VCC), U10.14 (VCC), U11.14 (VCC), U12.14 (VCC), U13.14 (VCC), U14.14 (VCC), U15.14 (VCC), U2.16 (VCC), U3.14 (VCC), U4.14 (VCC), U6.14 (VCC), U7.14 (VCC), U8.14 (VCC), U9.14 (VCC), 6-9(nice)1.2 (Vcc)
- net GND: now reaches U5.7 (GND)
- net GND: now also U1.8 (GND), U10.7 (GND), U11.7 (GND), U12.7 (GND), U13.7 (GND), U14.7 (GND), U15.7 (GND), U2.8 (GND), U3.7 (GND), U4.7 (GND), U6.7 (GND), U7.7 (GND), U8.7 (GND), U9.7 (GND), 6-9(nice)1.1 (Gnd)
- net at U11.12, U13.12, U3.12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: now also 6-9(nice)1.3 (Clk)
- net at U2.1 (A0): now also 6-9(nice)1.7 (Read_1)
- net at U2.2 (A1): now also 6-9(nice)1.8 (Read_2)
- net at U2.3 (A2): now also 6-9(nice)1.9 (Read_3)
- net at U2.4 (~{E1}): now also U1.4 (~{E1}), U1.5 (~{E2}), U2.5 (~{E2}), 6-9(nice)1.15 (Msc)
- net at U2.6 (E3): now also 6-9(nice)1.10 (Readable)
- net at U1.1 (A0): now also 6-9(nice)1.11 (Write_1)
- net at U1.2 (A1): now also 6-9(nice)1.12 (Write_2)
- net at U1.3 (A2): now also 6-9(nice)1.13 (Write_3)
- net at U1.6 (E3): now also 6-9(nice)1.14 (Writeable)

Commit message: im very bad
Changed lines of the file:
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@@
 		(on_board yes)
 		(dnp no)
-		(fields_autoplaced yes)
 		(property "Reference" "U5"
-			(at 152.0033 113.03 0)
+			(at 148.336 122.682 0)
 			(effects
 				(font
