File: pcbStuff/potato/v1/goodRAM/goodRAM.kicad_pcb (KiCad board)
At the start: 2 copper layers, 16 parts, among them U1 74HC238, U10 74LS74, U11 74LS08, U12 74LS74, U13 74LS08, U14 74LS74, U15 74LS74, U2 74HC238, U3 74LS08, U4 74LS74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

Commit message: im very bad
Parts:
- moved U8 146.4 mm to (152.4, 86.4), turned to 90 degrees
- moved U3 121.6 mm to (114.3, 86.4), turned to 90 degrees
- moved U5 118.7 mm to (128.3, 91.4)
- moved U4 117.2 mm to (115.6, 91.4)
- moved U7 112.0 mm to (141.0, 91.4)
- moved U6 111.0 mm to (133.3, 86.4), turned to 90 degrees
Routing:
- net Net-(6-9(nice)1-Bus_3): track 0.00 -> 128.9 mm, vias 0 -> 3
- net GND: track 0.00 -> 87.6 mm, vias 0 -> 7
- net Net-(6-9(nice)1-Bus_2): track 0.00 -> 68.7 mm, vias 0 -> 3
- net Net-(6-9(nice)1-Bus_1): track 0.00 -> 59.1 mm
- net Net-(6-9(nice)1-Clk): track 0.00 -> 40.2 mm
- net Net-(U5B-Q): track 0.00 -> 29.0 mm, vias 0 -> 2
- net Net-(U4B-Q): track 0.00 -> 21.2 mm
- net Net-(U7B-Q): track 0.00 -> 20.9 mm
- net Net-(U7A-Q): track 0.00 -> 20.6 mm
- net Net-(U5A-Q): track 0.00 -> 19.9 mm
- net Net-(U4A-Q): track 0.00 -> 15.8 mm, vias 0 -> 1
- net Net-(U2-Y4): track 0.00 -> 15.5 mm
- net Net-(U2-Y3): track 0.00 -> 15.5 mm
- net Net-(U5B-C): track 0.00 -> 14.3 mm
- net Net-(U4A-C): track 0.00 -> 12.5 mm

Commit message: DONE! ish
Parts:
- U1, U2: moved to B.Cu
- moved U13 178.1 mm to (190.5, 86.4), turned to 90 degrees
- moved U15 171.6 mm to (204.5, 91.4)
- moved U14 169.7 mm to (191.8, 91.4)
- moved U9 163.0 mm to (179.1, 91.4)
- moved U10 141.2 mm to (166.4, 91.4)
- moved U1 119.5 mm to (186.7, 64.8), turned to -90 degrees
- moved U11 116.6 mm to (152.4, 86.4), turned to 90 degrees
- moved U12 110.7 mm to (153.7, 91.4)
- moved U2 85.6 mm to (165.1, 64.8), turned to -90 degrees
- moved 6-9(nice)1 65.9 mm to (114.3, 64.8), turned to 90 degrees
- moved U8 19.0 mm to (171.4, 86.4)
Routing:
- net VCC: track 0.00 -> 300.3 mm, vias 0 -> 12
- net GND: track 87.6 -> 332.3 mm, vias 7 -> 8
- net Net-(6-9(nice)1-Bus_2): track 68.7 -> 249.2 mm, vias 3 -> 6
- net Net-(6-9(nice)1-Bus_3): track 128.9 -> 254.7 mm, vias 3 -> 12
- net Net-(6-9(nice)1-Bus_1): track 59.1 -> 157.6 mm, vias 0 -> 2
- net Net-(U1-Y3): track 0.00 -> 82.6 mm
- net Net-(6-9(nice)1-Write_1): track 0.00 -> 76.6 mm, vias 0 -> 1
- net Net-(6-9(nice)1-Write_2): track 0.00 -> 71.2 mm, vias 0 -> 1
- net Net-(U1-Y4): track 0.00 -> 66.1 mm
- net Net-(6-9(nice)1-Write_3): track 0.00 -> 65.1 mm, vias 0 -> 1
- net Net-(U2-Y7): track 0.00 -> 61.7 mm, vias 0 -> 1
- net Net-(6-9(nice)1-Clk): track 40.2 -> 94.4 mm
- net Net-(U2-Y3): track 15.5 -> 69.0 mm
- net Net-(6-9(nice)1-Writeable): track 0.00 -> 53.0 mm
- net Net-(U1-Y5): track 0.00 -> 49.6 mm
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Other:
- board outline added: 102.9 x 47 mm
- board text added: "RAM"

Commit message: PROGRESS FUCK YEAH
Routing:
- net Net-(U10A-C): track 12.5 -> 38.8 mm
- net Net-(U5B-C): track 15.5 -> 41.9 mm
- net Net-(U10B-C): track 15.5 -> 41.9 mm
- net Net-(U14A-C): track 15.0 -> 38.8 mm
- net Net-(U4A-C): track 23.5 -> 38.8 mm
- net Net-(6-9(nice)1-Bus_3): track 254.7 -> 269.7 mm
- net Net-(U5B-Q): track 29.0 -> 39.5 mm
- net Net-(U10B-Q): track 29.0 -> 39.5 mm
- net Net-(U5A-Q): track 19.9 -> 27.1 mm
- net Net-(U10A-Q): track 19.9 -> 27.1 mm
- net Net-(6-9(nice)1-Write_3): track 65.1 -> 67.6 mm
- net Net-(6-9(nice)1-Write_2): track 71.2 -> 73.7 mm
- net GND: track 332.3 -> 330.1 mm
- net VCC: track 300.3 -> 301.5 mm
- net Net-(6-9(nice)1-Bus_2): track 249.2 -> 248.1 mm
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Other:
- outline, holes or cut-outs redrawn
