File: pcbStuff/potato/v1/ALU/ALU.kicad_sch (KiCad schematic)
At the start: 10 parts, among them U1 74LS86, U2 74LS08, U3 74LS32, U4 74LS86, U5 74LS08, U6 74LS86, U7 74LS08, U8 74LS08, U9 74LS02

Commit message: wire
Parts:
- added U10, U11: 74LS02, symbol 74xx:74LS02
- added U12, U13, U14: 74LS74, symbol 74xx:74LS74
- added U15: 74LS08, symbol 74xx:74LS08
- added unit 3 of U7
- added unit 1 of U7
- added unit 2 of U7
- added unit 4 of U8
- added unit 5 of U8
Connections:
- net at U6.2: now also U13.5 (Q), U7.2
- net at U9.1, U9.5, U9.6: no longer U9.11, U9.12, U9.9
- net at U6.5: now also U12.9 (Q), U7.5
- net at U1.1, U2.1: now also U14.9 (Q), U15.2
- net at U9.10: now also U8.13
- net at U9.4, U9.8: now also U9.12
- net at U6.10: now also U12.5 (Q), U7.10
- net at U9.13: now also U9.9, U15.13
- new net: U10.1, U10.11, U10.12, U10.5, U10.6, U10.9, U11.3
- new net: U12.11 (C), U12.3 (C), U13.11 (C), U13.2 (D), U13.3 (C), U14.11 (C), U14.12 (D), U14.3 (C), U15.11, U15.3, U7.3, U8.11
- new net: U12.2 (D), U13.12 (D), U15.8, U7.8
- new net: U13.9 (Q), U15.10
- new net: U11.10, U11.11
- new net: U10.2, U11.8, U11.9
- new net: U12.12 (D), U14.2 (D), U15.6, U7.6
- new net: U14.5 (Q), U15.5
- new net: U10.4, U10.8
- new net: U11.12, U11.4
- new net: U7.1, U7.4, U7.9
- new net: U15.1, U15.4, U15.9
- new net: U11.1, U11.5, U11.6
- new net: U15.12, U8.12
- new net: U10.3, U11.2
- no-connect marks 1 -> 2
Other:
- moved on the sheet: U6D, U9A, U9B, U9C, U9D, U9E

Commit message: motivation stocks are tanking right now
Parts:
- removed U10, U11, U9: 74LS02, symbol 74xx:74LS02
- removed unit 3 of U3
- removed U5: 74LS08, symbol 74xx:74LS08
- added U10, U5: 74HC238, Package_DIP:DIP-16_W7.62mm, symbol 74xx:74HC238
- 6-9(nice)1: footprint (none) -> Connector_PinHeader_2.54mm:PinHeader_1x15_P2.54mm_Vertical
- U1, U12, U13, U14, U15, U2, U3, U4, U6, U7, U8: footprint (none) -> Package_DIP:DIP-14_W7.62mm
Connections:
- net GND: now also 6-9(nice)1.1 (Gnd), U12.7 (GND), U13.7 (GND), U14.7 (GND), U15.7 (GND), U7.14 (VCC), U8.7 (GND), U10.8 (GND), U5.8 (GND)
- net VCC: now also 6-9(nice)1.2 (Vcc), U12.14 (VCC), U13.14 (VCC), U14.14 (VCC), U15.14 (VCC), U7.7 (GND), U8.14 (VCC), U10.16 (VCC), U5.16 (VCC)
- net at U8.1, U8.4, U8.9: now also U5.13 (Y2)
- net at U8.3: now also 6-9(nice)1.4 (Bus_1), U12.11 (C), U12.3 (C), U13.11 (C), U13.2 (D), U13.3 (C), U14.11 (C), U14.12 (D), U14.3 (C), U15.11, U15.3, U7.3, U8.11
- net at U1.2, U6.3: now also U2.13; no longer U2.2
- net at U8.8: now also U12.2 (D), U13.12 (D), U15.8, U7.8
- net at U13.9 (Q), U15.10: now also U4.1
- net at 6-9(nice)1.10 (Readable): now also U5.6 (E3)
- net at 6-9(nice)1.11 (Write_1): now also U10.1 (A0)
- net at 6-9(nice)1.12 (Write_2): now also U10.2 (A1)
- net at 6-9(nice)1.13 (Write_3): now also U10.3 (A2)
- net at 6-9(nice)1.14 (Writeable): now also U10.6 (E3)
- net at 6-9(nice)1.3 (Clk): now also U15.12, U8.12
- net at 6-9(nice)1.5 (Bus_2): now also 6-9(nice)1.6 (Bus_3), U12.12 (D), U14.2 (D), U15.6, U7.6, U8.6
- net at 6-9(nice)1.7 (Read_1): now also U5.1 (A0)
- net at 6-9(nice)1.8 (Read_2): now also U5.2 (A1)
- net at 6-9(nice)1.9 (Read_3): now also U5.3 (A2)
- net at U1.10, U6.6: now also U2.5; no longer U2.10
- net at U2.8: now also U3.2; no longer U3.4
- net at U2.9: now also U1.3, U1.4; no longer U1.9
- net at U3.1: now also U2.11; no longer U2.3
- net at U2.6: now also U3.4; no longer U3.2
- net at U1.13, U3.3: now also U2.2; no longer U2.13
- net at U14.5 (Q), U15.5: now also U1.9, U2.4
- net at U7.1, U7.4, U7.9: now also U5.14 (Y1)
- net at U1.1, U14.9 (Q), U15.2: now also U2.12; no longer U2.1
- net at U15.1, U15.4, U15.9: now also U5.15 (Y0)
- net at U8.13: now also U10.14 (Y1)
- net at U15.13: now also U10.15 (Y0)
- net at U1.12, U1.8: now also U2.1; no longer U2.12
- net at U3.5: now also U2.3; no longer U2.11
- net at U1.5: now also U2.10; no longer U2.5
- no-connect marks 2 -> 1
Other:
- moved on the sheet: 6-9(nice)1, U12A, U12B, U12C, U13A, U13B, U13C, U14A, U14B, U14C, U15A, U15B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
