File: pcbStuff/keyboard/keyboard.kicad_sch (KiCad schematic)
At the start: 2 parts, among them SW1 SW_Push

Commit message: double reverse progress
Parts:
- removed D1: SK6812, LED_SMD:LED_SK6812_PLCC4_5.0x5.0mm_P3.2mm, symbol LED:SK6812
- removed SW1: SW_Push, Button_Switch_Keyboard:SW_Cherry_MX_1.00u_PCB, symbol Switch:SW_Push
- added A0: micro RIGHT, Connector_PinHeader_2.54mm:PinHeader_1x12_P2.54mm_Vertical, symbol Connector:Conn_01x12_Socket
- added A1: micro LEFT, Connector_PinHeader_2.54mm:PinHeader_1x12_P2.54mm_Vertical, symbol Connector:Conn_01x12_Socket
- added A3: micro BONUS, Connector_PinHeader_2.54mm:PinHeader_1x02_P2.54mm_Vertical, symbol Connector:Conn_01x02_Socket
Connections:
- new net COL0: A1.5 (Pin_5)
- new net COL1: A1.6 (Pin_6)
- new net COL2: A1.7 (Pin_7)
- new net COL3: A1.8 (Pin_8)
- new net COL4: A1.9 (Pin_9)
- new net COL5: A1.10 (Pin_10)
- new net COL6: A1.11 (Pin_11)
- new net COL7: A1.12 (Pin_12)
- new net COL8: A3.1 (Pin_1)
- new net GND: A1.2 (Pin_2)
- new net LED: A3.2 (Pin_2)
- new net ROW0: A0.1 (Pin_1)
- new net ROW1: A0.2 (Pin_2)
- new net ROW2: A0.5 (Pin_5)
- new net ROW3: A0.6 (Pin_6)
- new net ROW4: A0.7 (Pin_7)
- new net ROW5: A0.8 (Pin_8)
- new net ROW6: A0.9 (Pin_9)
- new net ROW7: A0.10 (Pin_10)
- new net ROW8: A0.11 (Pin_11)
- new net ROW9: A0.12 (Pin_12)
- new net VCC: A1.4 (Pin_4)

Commit message: not doing that right now
Parts:
- added D1, D10, D11, D12, D13, D14, D15, D16, D17, D18, D19, D2, D20, D21, D22, D23, D24, D25, D26, D27, D28, D29, D3, D30, D31, D32, D33, D34, D35, D36, D37, D38, D39, D4, D40, D41, D42, D43, D44, D45, D46, D47, D48, D49, D5, D50, D51, D52, D53, D54, D55, D56, D57, D58, D59, D6, D60, D61, D62, D63, D64, D65, D66, D67, D68, D69, D7, D70, D71, D72, D73, D74, D75, D76, D77, D78, D79, D8, D80, D81, D82, D83, D84, D85, D86, D9: 1N4148WT, Diode_SMD:D_SOD-523, symbol Diode:1N4148WT
- added SW1, SW10, SW11, SW12, SW13, SW14, SW15, SW16, SW17, SW18, SW19, SW2, SW20, SW21, SW22, SW23, SW24, SW25, SW26, SW27, SW28, SW29, SW3, SW30, SW31, SW32, SW33, SW34, SW35, SW36, SW37, SW38, SW39, SW4, SW40, SW41, SW42, SW43, SW44, SW45, SW46, SW47, SW48, SW49, SW5, SW50, SW51, SW52, SW53, SW54, SW55, SW56, SW57, SW58, SW59, SW6, SW60, SW61, SW62, SW63, SW64, SW65, SW66, SW67, SW68, SW69, SW7, SW70, SW71, SW72, SW73, SW74, SW75, SW76, SW77, SW78, SW79, SW8, SW80, SW81, SW82, SW83, SW84, SW85, SW86, SW9: button, Button_Switch_Keyboard:SW_Cherry_MX_1.00u_PCB, symbol Switch:SW_Push
Connections:
- net COL0: now also D1.2 (A), D16.2 (A), D17.2 (A), D32.2 (A), D33.2 (A), D48.2 (A), D49.2 (A), D62.2 (A), D76.2 (A), D86.2 (A)
- net COL1: now also D15.2 (A), D18.2 (A), D2.2 (A), D31.2 (A), D34.2 (A), D47.2 (A), D50.2 (A), D63.2 (A), D75.2 (A), D77.2 (A)
- net COL2: now also D14.2 (A), D19.2 (A), D3.2 (A), D30.2 (A), D35.2 (A), D46.2 (A), D51.2 (A), D64.2 (A), D78.2 (A), D85.2 (A)
- net COL3: now also D20.2 (A), D36.2 (A), D4.2 (A), D52.2 (A), D65.2 (A), D83.2 (A)
- net COL4: now also D21.2 (A), D37.2 (A), D5.2 (A), D53.2 (A), D66.2 (A), D74.2 (A), D82.2 (A), D84.2 (A)
- net COL5: now also D13.2 (A), D22.2 (A), D29.2 (A), D38.2 (A), D45.2 (A), D54.2 (A), D6.2 (A), D61.2 (A), D67.2 (A), D79.2 (A)
- net COL6: now also D10.2 (A), D23.2 (A), D26.2 (A), D39.2 (A), D42.2 (A), D55.2 (A), D58.2 (A), D68.2 (A), D7.2 (A), D71.2 (A)
- net COL7: now also D12.2 (A), D24.2 (A), D28.2 (A), D40.2 (A), D44.2 (A), D56.2 (A), D60.2 (A), D69.2 (A), D8.2 (A), D80.2 (A)
- net COL8: now also D11.2 (A), D25.2 (A), D27.2 (A), D41.2 (A), D43.2 (A), D57.2 (A), D59.2 (A), D70.2 (A), D72.2 (A), D73.2 (A), D81.2 (A), D9.2 (A)
- net ROW0: now also SW1.2, SW2.2, SW3.2, SW4.2, SW5.2, SW6.2, SW7.2, SW8.2, SW9.2
- net ROW1: now also SW17.2, SW18.2, SW19.2, SW20.2, SW21.2, SW22.2, SW23.2, SW24.2, SW25.2
- net ROW2: now also SW33.2, SW34.2, SW35.2, SW36.2, SW37.2, SW38.2, SW39.2, SW40.2, SW41.2
- net ROW3: now also SW49.2, SW50.2, SW51.2, SW52.2, SW53.2, SW54.2, SW55.2, SW56.2, SW57.2
- net ROW4: now also SW62.2, SW63.2, SW64.2, SW65.2, SW66.2, SW67.2, SW68.2, SW69.2, SW70.2
- net ROW5: now also SW71.2, SW76.2, SW77.2, SW78.2, SW79.2, SW80.2, SW81.2, SW82.2, SW83.2
- net ROW6: now also SW10.2, SW11.2, SW12.2, SW13.2, SW14.2, SW15.2, SW16.2
- net ROW7: now also SW26.2, SW27.2, SW28.2, SW29.2, SW30.2, SW31.2, SW32.2
- net ROW8: now also SW42.2, SW43.2, SW44.2, SW45.2, SW46.2, SW47.2, SW48.2, SW73.2, SW74.2
- net ROW9: now also SW58.2, SW59.2, SW60.2, SW61.2, SW72.2, SW75.2, SW84.2, SW85.2, SW86.2
- new net: D32.1 (K), SW32.1
- new net: D76.1 (K), SW76.1
- new net: D4.1 (K), SW4.1
- new net: D23.1 (K), SW23.1
- new net: D75.1 (K), SW75.1
- new net: D27.1 (K), SW27.1
- new net: D53.1 (K), SW53.1
- new net: D14.1 (K), SW14.1
- new net: D19.1 (K), SW19.1
- new net: D11.1 (K), SW11.1
- new net: D36.1 (K), SW36.1
- new net: D35.1 (K), SW35.1
- new net: D13.1 (K), SW13.1
- new net: D15.1 (K), SW15.1
- new net: D84.1 (K), SW84.1
- new net: D50.1 (K), SW50.1
- new net: D20.1 (K), SW20.1
- new net: D52.1 (K), SW52.1
- new net: D2.1 (K), SW2.1
- new net: D41.1 (K), SW41.1
- new net: D62.1 (K), SW62.1
- new net: D12.1 (K), SW12.1
- new net: D73.1 (K), SW73.1
- new net: D6.1 (K), SW6.1
- new net: D29.1 (K), SW29.1
- new net: D40.1 (K), SW40.1
- new net: D70.1 (K), SW70.1
- new net: D65.1 (K), SW65.1
- new net: D31.1 (K), SW31.1
- new net: D66.1 (K), SW66.1
- new net: D68.1 (K), SW68.1
- new net: D57.1 (K), SW57.1
- new net: D28.1 (K), SW28.1
- new net: D79.1 (K), SW79.1
- new net: D22.1 (K), SW22.1
- new net: D39.1 (K), SW39.1
- new net: D48.1 (K), SW48.1
- new net: D37.1 (K), SW37.1
- new net: D59.1 (K), SW59.1
- new net: D72.1 (K), SW72.1
- new net: D86.1 (K), SW86.1
- new net: D56.1 (K), SW56.1
- new net: D24.1 (K), SW24.1
- new net: D9.1 (K), SW9.1
- new net: D16.1 (K), SW16.1
- new net: D85.1 (K), SW85.1
- new net: D63.1 (K), SW63.1
- new net: D25.1 (K), SW25.1
- new net: D33.1 (K), SW33.1
- new net: D61.1 (K), SW61.1
- new net: D74.1 (K), SW74.1
- new net: D18.1 (K), SW18.1
- new net: D42.1 (K), SW42.1
- new net: D46.1 (K), SW46.1
- new net: D60.1 (K), SW60.1
- new net: D49.1 (K), SW49.1
- new net: D71.1 (K), SW71.1
- new net: D38.1 (K), SW38.1
- new net: D10.1 (K), SW10.1
- new net: D43.1 (K), SW43.1
- new net: D80.1 (K), SW80.1
- new net: D54.1 (K), SW54.1
- new net: D69.1 (K), SW69.1
- new net: D64.1 (K), SW64.1
- new net: D55.1 (K), SW55.1
- new net: D30.1 (K), SW30.1
- new net: D81.1 (K), SW81.1
- new net: D26.1 (K), SW26.1
- new net: D82.1 (K), SW82.1
- new net: D21.1 (K), SW21.1
- new net: D8.1 (K), SW8.1
- new net: D58.1 (K), SW58.1
- new net: D5.1 (K), SW5.1
- new net: D83.1 (K), SW83.1
- new net: D17.1 (K), SW17.1
- new net: D45.1 (K), SW45.1
- new net: D67.1 (K), SW67.1
- new net: D47.1 (K), SW47.1
- new net: D77.1 (K), SW77.1
- new net: D3.1 (K), SW3.1
- new net: D51.1 (K), SW51.1
- new net: D7.1 (K), SW7.1
- new net: D44.1 (K), SW44.1
- new net: D78.1 (K), SW78.1
- new net: D1.1 (K), SW1.1
- new net: D34.1 (K), SW34.1
Other:
- moved on the sheet: A0, A1, A3

Commit message: p[iofspojasdf
Parts:
- renumbered SW18 to !1, SW60 to "1, SW20 to #1, SW21 to $1, SW22 to %1, SW24 to &1, SW26 to (1, SW27 to )1, SW25 to *1, SW70 to ,1, SW28 to -1, SW71 to .1, SW72 to /1, SW59 to ;1, SW44 to =1, SW19 to @1, SW29 to BackSpace1, SW49 to CAPLock1, SW76 to Ctrl1, SW46 to DEL1, SW85 to Down1, SW1 to ESC1, SW47 to End1, SW61 to Enter1, SW2 to F1, SW11 to F10, SW12 to F11, SW13 to F12, SW3 to F2, SW4 to F3, SW5 to F4, SW6 to F5, SW7 to F6, SW8 to F7, SW9 to F8, SW10 to F9, SW31 to Home1, SW30 to Insert1, SW78 to LAlt1, SW77 to LMeta1, SW62 to LShift1, SW84 to Left1, SW15 to LockScreen1, SW48 to PGDN1, SW32 to PGUP1, SW16 to Pause1, SW14 to PrintScreen1, SW80 to RAlt1, SW83 to RCtrl1, SW81 to RMeta1, SW74 to RShift1, SW86 to Right1, SW79 to Space1, SW33 to Tab1, SW75 to Up1, SW73 to [1, SW45 to \1, SW82 to ]1, SW23 to ^1, SW17 to `1, SW50 to a2, SW67 to b1, SW65 to c1, SW52 to d87, SW36 to e1, SW53 to f13, SW54 to g1, SW55 to h1, SW41 to i1, SW56 to j1, SW57 to k1, SW58 to l1, SW69 to m1, SW68 to n1, SW42 to o1, SW43 to p1, SW34 to q1, SW37 to r1, SW51 to s1, SW38 to t1, SW40 to u1, SW66 to v1, SW35 to w1, SW64 to x1, SW39 to y1, SW63 to z1
