File: pcbStuff/keyboard/keyboard.kicad_pcb (KiCad board)
At the start: 2 copper layers, 175 parts, among them SW1 button, SW10 button, SW11 button, SW12 button, SW13 button, SW14 button, SW15 button, SW16 button, SW17 button, SW18 button, SW19 button, SW2 button, SW20 button, SW21 button, SW22 button, SW23 button, SW24 button, SW25 button, SW26 button, SW27 button, SW28 button, SW29 button, SW3 button, SW30 button, SW31 button, SW32 button, SW33 button, SW34 button, SW35 button, SW36 button, SW37 button, SW38 button, SW39 button, SW4 button, SW40 button, SW41 button, SW42 button, SW43 button, SW44 button, SW45 button, SW46 button, SW47 button, SW48 button, SW49 button, SW5 button, SW50 button, SW51 button, SW52 button, SW53 button, SW54 button, SW55 button, SW56 button, SW57 button, SW58 button, SW59 button, SW6 button, SW60 button, SW61 button, SW62 button, SW63 button, SW64 button, SW65 button, SW66 button, SW67 button, SW68 button, SW69 button, SW7 button, SW70 button, SW71 button, SW72 button, SW73 button, SW74 button, SW75 button, SW76 button, SW77 button, SW78 button, SW79 button, SW8 button, SW80 button, SW81 button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

Commit message: unplugged :(
Parts:
- D1, D12, D23: moved to F.Cu
- moved SW13 301.8 mm to (276.9, -154.9)
- moved SW2 298.8 mm to (257.8, -154.9)
- moved SW4 298.3 mm to (276.9, -97.8)
- moved SW45 270.8 mm to (276.9, -174.0)
- moved D23 268.2 mm to (238.1, -176.5)
- moved SW34 268.1 mm to (257.8, -174.0)
- moved D12 265.6 mm to (219.0, -176.5)
- moved SW23 265.0 mm to (238.8, -174.0)
- moved SW9 264.5 mm to (276.9, 54.6)
- moved SW36 263.9 mm to (276.9, -116.8)
- moved D1 263.0 mm to (200.0, -176.5)
- moved SW12 262.6 mm to (219.7, -174.0)
- moved SW25 260.8 mm to (257.8, -116.8)
- moved SW18 260.6 mm to (276.9, -2.54)
- moved SW27 260.4 mm to (276.9, -59.7)
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Routing:
- net Net-(D77-K): track 0.00 -> 2.54 mm
- net Net-(D68-K): track 0.00 -> 2.54 mm
- net Net-(D57-K): track 0.00 -> 2.54 mm
- net Net-(D46-K): track 0.00 -> 2.54 mm
- net Net-(D35-K): track 0.00 -> 2.54 mm
- net Net-(D24-K): track 0.00 -> 2.54 mm
- net Net-(D76-K): track 0.00 -> 2.54 mm
- net Net-(D65-K): track 0.00 -> 2.54 mm
- net Net-(D59-K): track 0.00 -> 2.54 mm
- net Net-(D54-K): track 0.00 -> 2.54 mm
- net Net-(D48-K): track 0.00 -> 2.54 mm
- net Net-(D43-K): track 0.00 -> 2.54 mm
- net Net-(D37-K): track 0.00 -> 2.54 mm
- net Net-(D26-K): track 0.00 -> 2.54 mm
- net Net-(D15-K): track 0.00 -> 2.54 mm
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
Commit message: p[iofspojasdf
Parts:
- moved k1 334.8 mm to (78.5, 146.9)
- moved ESC1 303.4 mm to (21.5, 70.9)
- moved D1 303.4 mm to (20.8, 68.4)
- moved D2 300.5 mm to (58.8, 68.4)
- moved F1 300.5 mm to (59.5, 70.9)
- moved D45 289.0 mm to (115.8, 64.0)
- moved \1 289.0 mm to (116.5, 66.5)
- moved D34 289.0 mm to (96.8, 64.0)
- moved q1 289.0 mm to (97.5, 66.5)
- moved D78 286.6 mm to (191.8, 125.4)
- moved LAlt1 286.6 mm to (192.5, 127.9)
- moved ^1 283.4 mm to (135.5, 89.9)
- moved D23 283.4 mm to (134.8, 87.4)
- moved D46 278.7 mm to (251.1, 140.0)
- moved DEL1 278.7 mm to (251.8, 142.5)
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- renumbered SW18 to !1, SW60 to "1, SW21 to $1, SW22 to %1, SW24 to &1, SW26 to (1, SW27 to )1, SW25 to *1, SW70 to ,1, SW28 to -1, SW71 to .1, SW72 to /1, SW59 to ;1, SW44 to =1, SW19 to @1, SW29 to BackSpace1, SW49 to CAPLock1, SW76 to Ctrl1, SW46 to DEL1, SW85 to Down1, SW1 to ESC1, SW47 to End1, SW61 to Enter1, SW2 to F1, SW11 to F10, SW12 to F11, SW13 to F12, SW3 to F2, SW4 to F3, SW5 to F4, SW6 to F5, SW7 to F6, SW8 to F7, SW9 to F8, SW10 to F9, SW31 to Home1, SW30 to Insert1, SW78 to LAlt1, SW77 to LMeta1, SW62 to LShift1, SW84 to Left1, SW15 to LockScreen1, SW48 to PGDN1, SW32 to PGUP1, SW16 to Pause1, SW14 to PrintScreen1, SW80 to RAlt1, SW83 to RCtrl1, SW81 to RMeta1, SW74 to RShift1, SW86 to Right1, SW79 to Space1, SW33 to Tab1, SW75 to Up1, SW73 to [1, SW45 to \1, SW82 to ]1, SW23 to ^1, SW17 to `1, SW50 to a2, SW67 to b1, SW65 to c1, SW52 to d87, SW36 to e1, SW53 to f13, SW54 to g1, SW55 to h1, SW41 to i1, SW56 to j1, SW57 to k1, SW58 to l1, SW69 to m1, SW68 to n1, SW42 to o1, SW43 to p1, SW34 to q1, SW37 to r1, SW51 to s1, SW38 to t1, SW40 to u1, SW66 to v1, SW35 to w1, SW64 to x1, SW39 to y1, SW63 to z1

Commit message: deep rock?
Parts:
- moved D57 420.1 mm to (77.8, 144.4)
- moved *1 320.9 mm to (173.5, 89.9)
- moved D25 320.9 mm to (172.8, 87.4)
- moved D33 191.0 mm to (20.8, 106.4)
- moved Tab1 191.0 mm to (21.5, 108.9)
- moved LMeta1 178.4 mm to (45.3, 165.9)
- moved D77 178.4 mm to (44.6, 163.4)
- moved %1 88.2 mm to (116.5, 89.9)
- moved D22 88.2 mm to (115.8, 87.4)
Changed lines of the file:
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@@
 	(footprint "Button_Switch_Keyboard:SW_Cherry_MX_1.00u_PCB"
 		(layer "F.Cu")
-		(at 191.35 21.59)
+		(at 21.54 108.92)
 		(descr "Cherry MX keyswitch, 1.00u, PCB mount, http://cherryamericas.com/wp-content/uploads/2014/12/mx_cat.pdf")
 		(tags "Cherry MX keyswitch 1.00u PCB")
@@
 	(footprint "Button_Switch_Keyboard:SW_Cherry_MX_1.00u_PCB"
 		(layer "F.Cu")
-		(at 172.3 21.59)
+		(at 116.54 89.92)
 		(descr "Cherry MX keyswitch, 1.00u, PCB mount, http://cherryamericas.com/wp-content/uploads/2014/12/mx_cat.pdf")
 		(tags "Cherry MX keyswitch 1.00u PCB")
@@
 	(footprint "Diode_SMD:D_SOD-523"
 		(layer "F.Cu")
-		(at 171.6 19.05 180)
+		(at 115.84 87.38 180)
 		(descr "http://www.diodes.com/datasheets/ap02001.pdf p.144")
 		(tags "Diode SOD523")
@@
 	(footprint "Diode_SMD:D_SOD-523"
 		(layer "F.Cu")
-		(at 171.6 38.1 180)
+		(at 44.59 163.38 180)
 		(descr "http://www.diodes.com/datasheets/ap02001.pdf p.144")
 		(tags "Diode SOD523")
@@
 	(footprint "Button_Switch_Keyboard:SW_Cherry_MX_1.00u_PCB"
 		(layer "F.Cu")
-		(at 229.45 -226.06)
+		(at 173.54 89.92)
 		(descr "Cherry MX keyswitch, 1.00u, PCB mount, http://cherryamericas.com/wp-content/uploads/2014/12/mx_cat.pdf")
 		(tags "Cherry MX keyswitch 1.00u PCB")
@@
 	(footprint "Diode_SMD:D_SOD-523"
 		(layer "F.Cu")
-		(at 228.75 -228.6 180)
+		(at 172.84 87.38 180)
 		(descr "http://www.diodes.com/datasheets/ap02001.pdf p.144")
 		(tags "Diode SOD523")
@@
 	(footprint "Button_Switch_Keyboard:SW_Cherry_MX_1.00u_PCB"
 		(layer "F.Cu")
-		(at 172.3 40.64)
+		(at 45.29 165.92)
 		(descr "Cherry MX keyswitch, 1.00u, PCB mount, http://cherryamericas.com/wp-content/uploads/2014/12/mx_cat.pdf")
 		(tags "Cherry MX keyswitch 1.00u PCB")
@@
 	(footprint "Diode_SMD:D_SOD-523"
 		(layer "F.Cu")
-		(at 190.65 19.05 180)
+		(at 20.84 106.38 180)
 		(descr "http://www.diodes.com/datasheets/ap02001.pdf p.144")
 		(tags "Diode SOD523")
@@
 	(footprint "Diode_SMD:D_SOD-523"
 		(layer "F.Cu")
-		(at 228.75 -247.65 180)
+		(at 77.84 144.38 180)
 		(descr "http://www.diodes.com/datasheets/ap02001.pdf p.144")
 		(tags "Diode SOD523")
@@
 	)
 	(segment
-		(start 172.3 19.05)
-		(end 172.3 21.59)
+		(start 116.54 87.38)
+		(end 116.54 89.92)
 		(width 0.2)
 		(layer "F.Cu")
@@
 	)
 	(segment
-		(start 229.45 -228.6)
-		(end 229.45 -226.06)
+		(start 173.54 87.38)
+		(end 173.54 89.92)
 		(width 0.2)
 		(layer "F.Cu")
@@
 	)
 	(segment
-		(start 191.35 19.05)
-		(end 191.35 21.59)
+		(start 21.54 106.38)
+		(end 21.54 108.92)
 		(width 0.2)
 		(layer "F.Cu")
@@
 	)
 	(segment
-		(start 229.45 -247.65)
-		(end 229.45 -245.11)
+		(start 78.54 144.38)
+		(end 78.54 146.92)
 		(width 0.2)
 		(layer "F.Cu")
@@
 	)
 	(segment
-		(start 172.3 38.1)
-		(end 172.3 40.64)
+		(start 45.29 163.38)
+		(end 45.29 165.92)
 		(width 0.2)
 		(layer "F.Cu")
@@
 	)
 	(group ""
+		(members "48bb4a4c-0bea-4ed5-aeae-7048217b91f5" "608b6d8f-2b64-4461-a7fa-a307b05bd8ac"
+			"67563e59-e6c1-43d1-a0d4-228cea45caca"
+		)
+	)
+	(group ""
 		(members "32669e80-4b90-4b41-b4ac-4448258898fe" "54ec9b81-9f5a-4a24-8e51-679f728567a0"
 			"73aad6bf-bfc3-4382-97c6-829413dee514"
@@
 	)
 	(group ""
+		(members "8c5234a1-7dc1-4d67-8ce6-e7f4a759a484" "9b6c2284-b3e0-4741-a38a-0e43b40f103f"
+			"eaf6944b-613b-430d-81d0-98c5adaa1fba"
+		)
+	)
+	(group ""
+		(members "5901adf9-0458-4d36-acde-744c4ef6bfe7" "61dc7c59-f255-4cac-a6ed-fd339a22bbba"
+			"8a344a13-a54e-44f1-bdb4-018b5c2d0894"
+		)
+	)
+	(group ""
+		(members "4edee1b5-7b8f-47a3-b3f1-aabecc59e115" "8bd55654-21a3-4237-bdbf-41acf166ee34"
+			"a7d1f79c-8d9a-4377-9ff2-b4c8a891e9e1"
+		)
+	)
+	(group ""
 		(members "1e6d2124-5a31-49af-8460-39ab870d154f" "40b41c3e-85c3-419e-9e33-29506f043c55"
 			"e74d1d81-699a-44c5-b7d5-642f3aaba9c6"
@@
 	)
 	(group ""
+		(members "53885a48-65d0-4a15-b7ff-728ba11ed7a0" "c7070312-3823-40b2-b9b9-fc0904505df6"
+			"e30370c1-cc29-438e-8caf-cb0da9d9d83e"
+		)
+	)
+	(group ""
 		(members "1f37b553-4b97-46be-9caa-e6053d4298d5" "7345d8db-e103-42ca-88a5-6f1bc5ebecae"
 			"ccb267eb-7af8-491e-9594-6ab1a0feb2d1"
@@
 		)
 	)
+	(group ""
+		(members "382835b8-76b6-4481-b8b6-d92e0676919b" "c320d679-7e0a-466c-abb7-17c2753222cb"
+			"d9147e82-615f-4af4-81d9-597c6b56793f"
+		)
+	)

Commit message: wawawewe
Parts:
- moved F11 244.9 mm to (534.2, 52.6)
- moved F12 244.9 mm to (553.2, 52.6)
- moved &1 244.9 mm to (456.0, 95.0)
- moved *1 244.9 mm to (418.0, 76.0)
- moved D2 244.9 mm to (303.3, 54.5)
- moved D22 244.9 mm to (360.3, 73.5)
- moved D23 244.9 mm to (379.3, 73.5)
- moved D24 244.9 mm to (455.3, 92.5)
- moved D25 244.9 mm to (417.3, 73.5)
- moved D3 244.9 mm to (322.3, 54.5)
- moved D33 244.9 mm to (265.3, 92.5)
- moved D34 244.9 mm to (341.3, 50.0)
- moved D35 244.9 mm to (398.3, 92.5)
- moved D45 244.9 mm to (360.3, 50.0)
- moved D56 244.9 mm to (398.3, 49.7)
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