File: pcbStuff/bongos/bongos.kicad_pcb (KiCad board)
At the start: 2 copper layers, 42 parts, among them SW1 SW_Push, SW2 SW_Push, SW3 SW_Push, SW4 SW_Push, SW5 SW_Push, U1 74LS04, U10 74LS04, U11 74LS74, U12 74LS74, U13 LM555xN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

Commit message: poor mans factorio
Parts:
- moved U10 91.2 mm to (82.5, 125.1), turned to -90 degrees
- moved U3 22.9 mm to (87.6, 93.3)
- moved U1 1.27 mm to (67.3, 99.1)
- moved U14 1.27 mm to (82.5, 114.3)
- moved U2 1.27 mm to (67.3, 110.5)
Routing:
- net Net-(R8-Pad2): track 6.43 -> 135.7 mm, vias 0 -> 7
- net Net-(R7-Pad2): track 6.43 -> 105.2 mm, vias 0 -> 5
- net Net-(R6-Pad2): track 6.43 -> 100.7 mm, vias 0 -> 4
- net Net-(R5-Pad2): track 6.35 -> 94.8 mm, vias 0 -> 5
- net GND: track 53.3 -> 116.7 mm, vias 0 -> 1
- net Net-(U2-Pad8): track 0.00 -> 32.7 mm, vias 0 -> 4
- net Net-(U2-Pad6): track 0.00 -> 22.3 mm, vias 0 -> 3
- net Net-(U1-Pad8): track 0.00 -> 13.5 mm, vias 0 -> 1
- net Net-(U1-Pad6): track 0.00 -> 13.3 mm, vias 0 -> 1
- net VCC: track 90.1 -> 103.1 mm
- net Net-(U14-Pad10): track 0.00 -> 11.6 mm, vias 0 -> 1
- net Net-(U14-Pad6): track 0.00 -> 7.62 mm
- net Net-(U2-Pad2): track 0.00 -> 2.54 mm
- net Net-(U2-Pad11): track 0.00 -> 2.54 mm
- net Net-(U2-Pad10): track 0.00 -> 2.54 mm
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
Commit message: gotta take breaks
Parts:
- moved U5 138.1 mm to (106.7, 149.2), turned to -90 degrees
- moved U15 135.8 mm to (165.1, 143.5), turned to -90 degrees
- moved U4 131.4 mm to (106.7, 139.1), turned to -90 degrees
- moved U9 120.2 mm to (130.8, 134.0), turned to -90 degrees
- moved U6 118.6 mm to (91.4, 136.5), turned to 90 degrees
- moved R1 110.4 mm to (71.8, 124.5), turned to -90 degrees
- moved R2 106.9 mm to (68.6, 124.5), turned to -90 degrees
- moved U7 104.4 mm to (91.4, 126.4), turned to 90 degrees
- moved U12 99.7 mm to (82.5, 144.8), turned to -90 degrees
- moved U11 95.8 mm to (82.5, 134.6), turned to -90 degrees
- moved U17 94.5 mm to (150.5, 109.9), turned to -90 degrees
- moved U10 76.1 mm to (151.1, 158.1)
- moved U13 72.6 mm to (82.5, 124.5), turned to -90 degrees
- moved C1 62.1 mm to (64.1, 126.9), turned to 90 degrees
Connections:
- U15 pad 3: Net-(U5B-~{R}) -> Net-(U4B-~{R})
- U15 pad 6: Net-(U5A-~{R}) -> Net-(U5B-~{R})
- U15 pad 8: Net-(U4B-~{R}) -> Net-(U5A-~{R})
- U17 pad 1: Net-(U4B-C) -> Net-(U5A-C)
- U17 pad 10: Net-(U17-Pad10) -> unconnected-(U17-Pad10)
- U17 pad 11: unconnected-(U17-Pad11) -> Net-(U10-Pad11)
- U17 pad 12: unconnected-(U17-Pad12) -> Net-(U17-Pad12)
- U17 pad 13: unconnected-(U17-Pad13) -> Net-(U17-Pad13)
- U17 pad 3: Net-(U17-Pad10) -> Net-(U17-Pad13)
- U17 pad 4: Net-(U5B-C) -> Net-(U4B-C)
- U17 pad 5: Net-(U5A-C) -> Net-(U5B-C)
- U17 pad 6: Net-(U17-Pad6) -> Net-(U17-Pad12)
- U17 pad 8: Net-(U10-Pad11) -> unconnected-(U17-Pad8)
- U17 pad 9: Net-(U17-Pad6) -> unconnected-(U17-Pad9)
- U3 pad 11: Net-(U5B-C) -> Net-(U4B-C)
- U3 pad 6: Net-(U4B-C) -> Net-(U5A-C)
- U3 pad 8: Net-(U5A-C) -> Net-(U5B-C)
- U4 pad 12: Net-(U11A-~{S}) -> Net-(U11A-D)
- U4 pad 9: Net-(D2-A) -> Net-(D4-A)
- U5 pad 12: Net-(U11A-D) -> Net-(U12A-D)
- U5 pad 2: Net-(U12A-D) -> Net-(U11A-~{S})
- U5 pad 5: Net-(D3-A) -> Net-(D2-A)
- U5 pad 9: Net-(D4-A) -> Net-(D3-A)
- U6 pad 1: Net-(U4A-~{Q}) -> Net-(U4A-C)
- U6 pad 10: Net-(U5A-C) -> Net-(U5B-C)
- U6 pad 12: Net-(U5B-~{Q}) -> Net-(U4B-~{Q})
- U6 pad 13: Net-(U5B-C) -> Net-(U4B-C)
- U6 pad 2: Net-(U4A-C) -> Net-(U4A-~{Q})
- U6 pad 4: Net-(U4B-~{Q}) -> Net-(U5A-~{Q})
- U6 pad 5: Net-(U4B-C) -> Net-(U5A-C)
- U6 pad 9: Net-(U5A-~{Q}) -> Net-(U5B-~{Q})
- U7 pad 1: Net-(D1-A) -> Net-(U4B-C)
- U7 pad 11: Net-(U15-Pad2) -> Net-(U4A-~{R})
- U7 pad 12: Net-(D4-A) -> Net-(D1-A)
- U7 pad 13: Net-(U5B-C) -> Net-(U4A-C)
- U7 pad 2: Net-(U4A-C) -> Net-(D4-A)
- U7 pad 3: Net-(U4A-~{R}) -> Net-(U15-Pad2)
- U7 pad 4: Net-(D2-A) -> Net-(D3-A)
- U7 pad 5: Net-(U4B-C) -> Net-(U5B-C)
- U7 pad 6: Net-(U15-Pad10) -> Net-(U15-Pad5)
- U7 pad 8: Net-(U15-Pad5) -> Net-(U15-Pad10)
- U7 pad 9: Net-(D3-A) -> Net-(D2-A)
- U8 pad 10: Net-(U8-Pad10) -> Net-(U10-Pad8)
- U8 pad 11: Net-(U10-Pad1) -> Net-(U8-Pad11)
- U8 pad 13: Net-(U10-Pad8) -> Net-(U8-Pad13)
- U8 pad 3: Net-(U8-Pad10) -> Net-(U8-Pad13)
- U8 pad 6: Net-(U8-Pad6) -> Net-(U8-Pad12)
- U8 pad 8: Net-(U8-Pad12) -> Net-(U10-Pad1)
- U8 pad 9: Net-(U8-Pad6) -> Net-(U8-Pad11)
Routing:
- net Net-(U5A-C): track 0.00 -> 96.9 mm, vias 0 -> 4
- net Net-(U5B-C): track 0.00 -> 86.4 mm, vias 0 -> 3
- net VCC: track 103.1 -> 179.9 mm, vias 0 -> 2
- net Net-(U4A-C): track 0.00 -> 75.2 mm, vias 0 -> 4
- net Net-(U11A-~{S}): track 0.00 -> 70.4 mm, vias 0 -> 2
- net Net-(U4B-C): track 0.00 -> 69.1 mm, vias 0 -> 3
- net Net-(U11A-D): track 0.00 -> 62.3 mm, vias 0 -> 3
- net Net-(U11A-C): track 0.00 -> 55.5 mm, vias 0 -> 2
- net Net-(U12A-D): track 0.00 -> 43.3 mm, vias 0 -> 1
- net Net-(U11A-Q): track 0.00 -> 42.0 mm, vias 0 -> 2
- net GND: track 116.7 -> 143.1 mm
- net Net-(R7-Pad2): track 105.2 -> 81.7 mm, vias 5 -> 4
- net Net-(U13-DIS): track 0.00 -> 23.2 mm, vias 0 -> 2
- net Net-(R8-Pad2): track 135.7 -> 116.4 mm, vias 7 -> 5
- net Net-(U13-THR): track 0.00 -> 15.6 mm, vias 0 -> 1
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
Commit message: fable foo
Parts:
- moved U8 102.7 mm to (110.5, 119.4), turned to 90 degrees
- moved U10 78.6 mm to (97.8, 100.3), turned to 0 degrees
- moved U9 42.5 mm to (123.8, 92.1)
- moved SW5 25.9 mm to (98.4, 92.7)
- moved U17 17.6 mm to (137.2, 98.4), turned to 0 degrees
- moved R1 1.27 mm to (71.8, 125.7)
- moved R2 1.27 mm to (68.6, 125.7)
- moved U12 1.27 mm to (82.5, 146.1)
- moved U13 1.27 mm to (82.5, 125.7)
- moved U11 1.27 mm to (82.5, 135.9)
Connections:
- U10 pad 1: Net-(U10-Pad1) -> Net-(R4-Pad2)
- U10 pad 12: unconnected-(U10-Pad12) -> Net-(U9A-~{S})
- U10 pad 13: unconnected-(U10-Pad13) -> Net-(U10-Pad13)
- U10 pad 2: Net-(U9A-~{S}) -> Net-(U11A-~{S})
- U10 pad 3: Net-(U10-Pad3) -> unconnected-(U10-Pad3)
- U10 pad 4: Net-(U13-R) -> unconnected-(U10-Pad4)
- U10 pad 5: Net-(R4-Pad2) -> Net-(U10-Pad5)
- U10 pad 6: Net-(U11A-~{S}) -> Net-(U13-R)
- U14 pad 8: Net-(U10-Pad3) -> Net-(U10-Pad5)
- U8 pad 8: Net-(U10-Pad1) -> Net-(U10-Pad13)
Routing:
- net Net-(U10-Pad5): track 0.00 -> 38.3 mm
- net Net-(U13-R): track 0.00 -> 32.3 mm, vias 0 -> 1
- net Net-(U11A-~{S}): track 70.4 -> 101.3 mm
- net GND: track 143.1 -> 162.8 mm, vias 1 -> 2
- net VCC: track 179.9 -> 190.6 mm
- net Net-(R4-Pad2): track 0.00 -> 3.38 mm
- net Net-(U5A-C): track 96.9 -> 98.3 mm
- net Net-(U13-THR): track 15.6 -> 16.9 mm, vias 1 -> 0
